File: Magnetic_FlowMeter/_autosave-Magnetic_FlowMeter.kicad_pcb (KiCad board)
At the start: 2 copper layers, 101.6 x 53.3 mm, 13 parts, among them P1 Digital, P10 CONN_01X01, P11 CONN_01X01, P12 CONN_01X01, P13 CONN_01X01, P2 Power, P3 Analog, P4 Analog, P5 PWM, P6 PWM, P7 Communication, P8 CONN_01X01, P9 CONN_01X01

Commit message: Update
Parts:
- added REF**: LCD-016N002L, Displays:LCD-016N002L, F.Cu at (241.3, 120.7)
- moved P10 91.4 mm to (276.1, 69.6)
- moved P11 91.4 mm to (194.8, 21.3)
- moved P12 91.4 mm to (245.6, 36.6)
- moved P13 91.4 mm to (269.7, 21.3)
- moved P2 91.4 mm to (207.5, 69.6)
- moved P3 91.4 mm to (230.4, 69.6)
- moved P4 91.4 mm to (253.2, 69.6)
- moved P5 91.4 mm to (198.4, 21.3)
- moved P6 91.4 mm to (225.3, 21.3)
- moved P7 91.4 mm to (248.2, 21.3)
- moved P8 91.4 mm to (193.5, 69.6)
- moved P1 91.4 mm to (273.6, 64.5)
- moved P9 91.4 mm to (245.6, 64.5)
