File: Magnetic_FlowMeter/_saved_Magnetic_FlowMeter.sch (KiCad schematic (older format))
At the start: 31 parts, among them P1 Digital, P10 CONN_01X01, P11 CONN_01X01, P12 CONN_01X01, P13 CONN_01X01, P2 Power, P3 Analog, P4 Analog, P5 PWM, P6 PWM, P7 Communication, P8 CONN_01X01, P9 CONN_01X01

Commit message: Update
Parts:
- removed 0.1uF (x5), 1uF (x4), 270pF (x2), 680pF: C, symbol C
- removed 10uF (x2): CP1, symbol CP1
- removed R10 (x2): R, symbol R
- removed U?: AD813, symbol AD813
- removed U?: AD7171, Housings_DFN_QFN:DFN-10-1EP_3x3mm_Pitch0.5mm, symbol AD7171
- added DS2: LCD-016N002L, WC1602A, symbol LCD-016N002L
- added R220: R, symbol R
- added RV12: POT_Dual_Separate, symbol POT_Dual_Separate
Connections:
- wire segments 126 -> 125
